Commit message: velodyne or laserscan 사용하여 map->odom->base_link 트리 만들어짐. ( visual odom 은 아직 적용 안되었음 )

File: description/robot.urdf.xacro (robot description, xacro)
@@ -33,3 +33,9 @@
     <origin xyz="0 0 0" rpy="0 0 0" />
   </joint>
+  <link name="camera_link"></link>
+  <joint name="camera_joint" type="fixed">
+    <parent link="base_link"/>
+    <child link="camera_link" />
+    <origin xyz="0 0 0" rpy="0 0 0" />
+  </joint>
 </robot>

Commit message: velodyne lidar + 3gx IMU 사용한 버전

File: description/robot.urdf.xacro (robot description, xacro)
@@ -13,5 +13,5 @@
     <parent link="chassis_link" />
     <child link="imu_link" />
-    <origin xyz="0 0 0" rpy="0 0 0" />
+    <origin xyz="0 0 0.15" rpy="0 0 0" />
   </joint>
   <link name="velodyne"> </link>
@@ -19,5 +19,5 @@
     <parent link="chassis_link" />
     <child link="velodyne" />
-    <origin xyz="0 0 0" rpy="0 0 0" />
+    <origin xyz="0.4 0 0.3" rpy="0 0 0" />
   </joint>
   <link name="navsat_link"> </link>

Commit message: cartographer lidar+imu+odom

File: description/robot.urdf.xacro (robot description, xacro)
@@ -2,4 +2,10 @@
 <robot name="lio" xmlns:xacro="http://tixiaoshan.github.io/">
   <xacro:property name="PI" value="3.1415926535897931" />
+  <link name="camera_pose_frame"></link>
+  <joint name="camera_pose_joint" type="fixed">
+    <parent link="camera_pose_frame"/>
+    <child link="base_link" />
+    <origin xyz="0 0 0" rpy="0 0 0" />
+  </joint>
   <link name="chassis_link"></link>
   <link name="base_link"></link>
@@ -37,5 +43,11 @@
     <parent link="base_link"/>
     <child link="camera_link" />
+    <origin xyz="0.4 0 0.15" rpy="0 0 0" />
+  </joint>
+<!--
+  <joint name="camera_pose_joint" type="fixed">
+    <parent link="camera_link"/>
+    <child link="camera_pose_frame" />
     <origin xyz="0 0 0" rpy="0 0 0" />
-  </joint>
+  </joint> -->
 </robot>
